File: Circuit Design/Kicad/SB_Hub_IF/SB_Hub_IF.kicad_pcb (KiCad board)
At the start: 4 copper layers, 69.7 x 76.8 mm, 56 parts, among them J1 POWER, J2 COMPUTER, U1 MCP23008-xSO

Commit message: Reorganised
Parts:
- removed C12: 1µ, MS_Favourites:Cap_THT_1µF_polarised
- removed LM1: LM1117, Package_TO_SOT_SMD:SOT-223-3_TabPin2
- removed R10, R11, R12, R13, R14, R5, R6, R8, R9: 10K, MS_Favourites:Resistor_SMD_1206_HandSolder
- removed R4: 1K, MS_Favourites:Resistor_SMD_1206_HandSolder
- C1, C11, C14: value 1µ -> 4.7µ
- J2: value COMPUTER -> HOST
- R1: value 1K -> 100R
- R3, R7: value 22K -> 10K
- SB2: value Dev2 -> Dev1
- SB3: value Dev3 -> Dev1
- SB4: value Dev4 -> Dev1
- SB5: value Dev5 -> Dev1
- SB6: value Dev6 -> Dev1
- SB7: value Dev7 -> Dev1
- SB8: value Dev8 -> Dev1
- moved D1 25.0 mm to (104.7, 100.4)
- moved R19 25.0 mm to (104.7, 94.2)
- moved J1 18.9 mm to (121.1, 108.4)
- moved C2 16.7 mm to (127.9, 104.4)
- moved C1 12.7 mm to (121.5, 101.1)
- moved R1 12.3 mm to (164.9, 105.1)
- moved R16 11.1 mm to (129.9, 99.2), turned to 180 degrees
- moved J2 10.6 mm to (161.8, 114.6)
- moved H2 9.53 mm to (111.7, 100.0)
- moved H6 9.53 mm to (160.9, 100.0)
- moved R2 9.43 mm to (154.1, 105.5)
- moved R20 9.43 mm to (151.5, 105.5)
- moved R15 9.24 mm to (147.8, 99.3)
- moved G*** 8.56 mm to (107.0, 107.9)
- moved C13 7.52 mm to (129.9, 94.8), turned to 180 degrees
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Connections:
- C13 pad 1: +3V3 -> +5V
- J2 pad 1: /~{SB_INT} -> GND
- J2 pad 2: /SB_CLK -> /SB_CLKH
- J2 pad 4: /SCL -> GND
- J2 pad 5: /SDA -> /SCL
- J2 pad 6: GND -> /SDA
- R1 pad 1: /CLK -> /SB_CLK
- R1 pad 2: /SB_CLK -> /SB_CLKH
- R15 pad 2: +3V3 -> +5V
- R16 pad 2: +3V3 -> +5V
- R17 pad 2: +3V3 -> +5V
- R18 pad 2: +3V3 -> +5V
- R19 pad 2: +3V3 -> +5V
- R2 pad 2: +3V3 -> +5V
- R20 pad 2: +3V3 -> +5V
- R3 pad 1: /CLK -> /SB_CLK
- R3 pad 2: +3V3 -> +5V
- R7 pad 2: +3V3 -> +5V
- SB1 pad 3: /CLK -> /SB_CLK
- SB1 pad 4: /~{INT} -> GND
- SB1 pad 5: /~{SB_ACT} -> DAT1
- SB1 pad 6: DAT1 -> /~{SB_ACT}
- SB2 pad 3: /CLK -> /SB_CLK
- SB2 pad 4: /~{INT} -> GND
- SB2 pad 5: /~{SB_ACT} -> DAT2
- SB2 pad 6: DAT2 -> /~{SB_ACT}
- SB3 pad 3: /CLK -> /SB_CLK
- SB3 pad 4: /~{INT} -> GND
- SB3 pad 5: /~{SB_ACT} -> DAT3
- SB3 pad 6: DAT3 -> /~{SB_ACT}
- SB4 pad 3: /CLK -> /SB_CLK
- SB4 pad 4: /~{INT} -> GND
- SB4 pad 5: /~{SB_ACT} -> DAT4
- SB4 pad 6: DAT4 -> /~{SB_ACT}
- SB5 pad 3: /CLK -> /SB_CLK
- SB5 pad 4: /~{INT} -> GND
- SB5 pad 5: /~{SB_ACT} -> DAT5
- SB5 pad 6: DAT5 -> /~{SB_ACT}
- SB6 pad 3: /CLK -> /SB_CLK
- SB6 pad 4: /~{INT} -> GND
- SB6 pad 5: /~{SB_ACT} -> DAT7
- SB6 pad 6: DAT6 -> /~{SB_ACT}
- SB7 pad 3: /CLK -> /SB_CLK
- SB7 pad 4: /~{INT} -> GND
- SB7 pad 5: /~{SB_ACT} -> DAT6
- SB7 pad 6: DAT7 -> /~{SB_ACT}
- SB8 pad 3: /CLK -> /SB_CLK
- SB8 pad 4: /~{INT} -> GND
- SB8 pad 5: /~{SB_ACT} -> DAT8
- SB8 pad 6: DAT8 -> /~{SB_ACT}
- U1 pad 18: +3V3 -> +5V
Routing:
- net /~{INT}: track 211.6 -> 0.00 mm, vias 2 -> 0
- net /CLK: track 210.9 -> 0.00 mm, vias 1 -> 0
- net /SB_CLK: track 8.56 -> 205.1 mm
- net +3V3: track 72.7 -> 0.00 mm, vias 23 -> 0
- net GND: track 3.25 -> 41.1 mm, vias 37 -> 42
- net /~{SB_ACT}: track 220.9 -> 205.6 mm, vias 1 -> 0
- net DAT6: track 30.2 -> 15.4 mm
- net /SB_CLKH: track 0.00 -> 10.3 mm
- net /~{SB_INT}: track 10.1 -> 0.00 mm
- net DAT7: track 20.7 -> 28.2 mm, vias 0 -> 2
- net Net-(JP1-C): track 7.35 -> 13.6 mm
- net DAT3: track 37.7 -> 31.5 mm, vias 1 -> 0
- net DAT5: track 41.7 -> 44.8 mm, vias 1 -> 0
- net Net-(JP3-C): track 6.47 -> 3.73 mm
- net Net-(JP2-C): track 11.7 -> 8.95 mm
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- added copper zone on In2.Cu, net +5V
- added copper zone on B.Cu, net GND
- added copper zone on In1.Cu, net GND
- removed copper zone on In1.Cu, net +3V3
- removed copper zone on B.Cu, net +5V
- removed copper zone on In2.Cu, net GND
Other:
- board size 69.7 x 76.8 mm -> 69.7 x 66.3 mm
- board text added: "SensorBus Hub I/F Rev A.1 Nov 2025"
- board text removed: "Sensor Bus Hub I/F Rev A.1 Sept 2025"
- board text removed: "~{INT}"
