File: Circuit Design/Kicad/SB_Hub_IF/SB_Hub_IF.kicad_sch (KiCad schematic)
At the start: 55 parts, among them J1 POWER, J2 COMPUTER, U1 MCP23008-xSO

Commit message: Tidy up
Parts:
- C1, C11, C14: value 1µ -> 4.7µ
Other:
- moved on the sheet: C1, C10, C11, C12, C14, C2, C3, C4, C5, C6, C7, C8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

Commit message: Reorganised
Parts:
- removed C12: 1µ, MS_Favourites:Cap_THT_1µF_polarised, symbol Device:C
- removed LM1: LM1117, Package_TO_SOT_SMD:SOT-223-3_TabPin2, symbol MS_Power:LM1117
- removed R10, R11, R12, R13, R14, R5, R6, R8, R9: 10K, MS_Favourites:Resistor_SMD_1206_HandSolder, symbol Device:R
- removed R4: 1K, MS_Favourites:Resistor_SMD_1206_HandSolder, symbol Device:R
- J2: value COMPUTER -> HOST
- R1: value 1K -> 100R
- R3, R7: value 22K -> 10K
- SB2: value Dev2 -> Dev1
- SB3: value Dev3 -> Dev1
- SB4: value Dev4 -> Dev1
- SB5: value Dev5 -> Dev1
- SB6: value Dev6 -> Dev1
- SB7: value Dev7 -> Dev1
- SB8: value Dev8 -> Dev1
Connections:
- net +3V3 is gone; now on net +5V: C13.1, R15.2, R16.2, R17.2, R18.2, R19.2, R2.2, R20.2, R3.2, R7.2, U1.18 (VDD)
- net CLK is gone; now on net SB_CLK: R1.1, R3.1, SB1.3 (CLK), SB2.3 (CLK), SB3.3 (CLK), SB4.3 (CLK), SB5.3 (CLK), SB6.3 (CLK), SB7.3 (CLK), SB8.3 (CLK)
- net ~{INT} is gone; now on net GND: SB1.4 (GND), SB2.4 (GND), SB3.4 (GND), SB4.4 (GND), SB5.4 (GND), SB6.4 (GND), SB7.4 (GND), SB8.4 (GND)
- net ~{SB_INT} is gone; now on net GND: J2.1 (Pin_1)
- net DAT1: now also SB1.5 (DAT); no longer SB1.6 (DAT)
- net DAT2: now also SB2.5 (DAT); no longer SB2.6 (DAT)
- net DAT3: now also SB3.5 (DAT); no longer SB3.6 (DAT)
- net DAT4: now also SB4.5 (DAT); no longer SB4.6 (DAT)
- net DAT5: now also SB5.5 (DAT); no longer SB5.6 (DAT)
- net DAT6: now also SB7.5 (DAT); no longer SB6.6 (DAT)
- net DAT7: now also SB6.5 (DAT); no longer SB7.6 (DAT)
- net DAT8: now also SB8.5 (DAT); no longer SB8.6 (DAT)
- net GND: now also J2.4 (Pin_4); no longer J2.6 (Pin_6)
- net SB_CLK: no longer J2.2 (Pin_2), R1.2
- net SCL: now also J2.5 (Pin_5); no longer J2.4 (Pin_4)
- net SDA: now also J2.6 (Pin_6); no longer J2.5 (Pin_5)
- net ~{SB_ACT}: now also SB1.6 (~{ACT}), SB2.6 (~{ACT}), SB3.6 (~{ACT}), SB4.6 (~{ACT}), SB5.6 (~{ACT}), SB6.6 (~{ACT}), SB7.6 (~{ACT}), SB8.6 (~{ACT}); no longer SB1.5 (~{ACT}), SB2.5 (~{ACT}), SB3.5 (~{ACT}), SB4.5 (~{ACT}), SB5.5 (~{ACT}), SB6.5 (~{ACT}), SB7.5 (~{ACT}), SB8.5 (~{ACT})
- new net SB_CLKH: J2.2 (Pin_2), R1.2
Other:
- moved on the sheet: D1, R1, R19, SB1
